Commit message: updated inverted URDF

File: fp_darc/urdf/fp_darc.urdf (robot description, URDF)
Before this commit: robot fp_darc, 5 links, 4 joints
Joints:
- joint base_footprint_base_link_joint: origin xyz=0.0 0.0 0.0 rpy=0.0 0.0 0.0 -> xyz=0.0 0.0 0.0 rpy=0.0 0.0 3.14159265359
- joint base_link_left_wheel_joint: origin xyz=0.1308 0.196 0.0325 rpy=-1.5707963267948966 -0.0 0.0 -> xyz=0.1308 0.196 0.0325 rpy=-1.5707963267948966 -0.0 3.14159265359
- joint base_link_lidar_joint: origin xyz=0.17920000000000003 0.0 0.23870000000000002 rpy=0.0 -0.0 0.0 -> xyz=0.17920000000000003 0.0 0.23870000000000002 rpy=0.0 -0.0 3.14159265359
- joint base_link_right_wheel_joint: origin xyz=0.1308 -0.196 0.0325 rpy=1.5707963267948966 -0.0 0.0 -> xyz=0.1308 -0.196 0.0325 rpy=1.5707963267948966 -0.0 3.14159265359

Commit message: created a single launch file

File: fp_darc/urdf/fp_darc.urdf (robot description, URDF)
Before this commit: robot fp_darc, 5 links, 4 joints
Joints:
- joint base_footprint_base_link_joint: origin xyz=0.0 0.0 0.0 rpy=0.0 0.0 3.14159265359 -> xyz=0.0 0.0 0.0 rpy=0.0 0.0 0.0
- joint base_link_left_wheel_joint: origin xyz=0.1308 0.196 0.0325 rpy=-1.5707963267948966 -0.0 3.14159265359 -> xyz=-0.1308 -0.196 0.0325 rpy=1.5707963267948966 -0.0 0.0
- joint base_link_lidar_joint: origin xyz=0.17920000000000003 0.0 0.23870000000000002 rpy=0.0 -0.0 3.14159265359 -> xyz=-0.17920000000000003 0.0 0.23870000000000002 rpy=0.0 -0.0 0.0
- joint base_link_right_wheel_joint: origin xyz=0.1308 -0.196 0.0325 rpy=1.5707963267948966 -0.0 3.14159265359 -> xyz=-0.1308 0.196 0.0325 rpy=-1.5707963267948966 -0.0 0.0

Commit message: updated code just beginning of corrected map

File: fp_darc/urdf/fp_darc.urdf (robot description, URDF)
Before this commit: robot fp_darc, 5 links, 4 joints
Joints:
- joint base_link_left_wheel_joint: origin xyz=-0.1308 -0.196 0.0325 rpy=1.5707963267948966 -0.0 0.0 -> xyz=0.1308 0.196 0.0325 rpy=-1.5707963267948966 -0.0 0.0
- joint base_link_lidar_joint: origin xyz=-0.17920000000000003 0.0 0.23870000000000002 rpy=0.0 -0.0 0.0 -> xyz=0.17920000000000003 0.0 0.23870000000000002 rpy=0.0 -0.0 0.0
- joint base_link_right_wheel_joint: origin xyz=-0.1308 0.196 0.0325 rpy=-1.5707963267948966 -0.0 0.0 -> xyz=0.1308 -0.196 0.0325 rpy=1.5707963267948966 -0.0 0.0
